Commit message: Add : Use Point to control Robot Arm, and use rviz for checking.

File: urdf/Robot_Arm.urdf (robot description, URDF)
Before this commit: robot Robot_Arm, 5 links, 4 joints
Joints:
- joint arm_joint_2: axis 0 1 0 -> 1 0 0
- joint arm_joint_3: axis 0 1 0 -> 1 0 0

Commit message: Add : Limit the Joint Angle.

File: urdf/Robot_Arm.urdf (robot description, URDF)
Before this commit: robot Robot_Arm, 5 links, 4 joints
Joints:
- joint arm_joint_2: axis 1 0 0 -> 0 1 0
- joint arm_joint_3: axis 1 0 0 -> 0 1 0

Commit message: Fix : Change the meshes to the current model.

File: urdf/Robot_Arm.urdf (robot description, URDF)
Before this commit: robot Robot_Arm, 5 links, 4 joints
Links:
- added link gripper_left; visual mesh filename=package://robot_arm_control/meshes/Gripper.stl scale=0.001 0.001 0.001
- added link gripper_right; visual mesh filename=package://robot_arm_control/meshes/Gripper.stl scale=-0.001 0.001 0.001
- link arm_link_1: geometry visual mesh filename=package://robot_arm_control/meshes/arm_link_1.stl scale=0.001 0.001 0.001
- link arm_link_2: geometry visual mesh filename=package://robot_arm_control/meshes/arm_link_2.stl scale=0.001 0.001 0.001
- link arm_link_3: geometry visual mesh filename=package://robot_arm_control/meshes/arm_link_3.stl scale=0.001 0.001 0.001
Joints:
- added joint Gripper_left: type continuous, parent arm_link_3, child gripper_left, origin xyz=-0.0175 0.015 0.064 rpy=0 0 0
- added joint Gripper_right: type continuous, parent arm_link_3, child gripper_right, origin xyz=-0.0175 -0.015 0.064 rpy=0 0 0
- joint arm_end_effector: origin xyz=0.0 0.0 0.13 rpy=0 0 0 -> xyz=0.0 0.0 0.123 rpy=0 0 0
- joint arm_joint_1: origin xyz=0.0 0.0 0.1 rpy=0 0 0 -> xyz=0.0 0.0 0.11 rpy=0 0 0
- joint arm_joint_2: origin xyz=0.0 0.0 0.20271 rpy=0 0 0 -> xyz=0.0 0.0 0.10 rpy=0 0 0
- joint arm_joint_3: origin xyz=0.0 0.0 0.269 rpy=0 0 0 -> xyz=0.0 0.0 0.17 rpy=0 0 0

Commit message: Add : Visualize the gripper animation, and change the msg to arduino.

File: urdf/Robot_Arm.urdf (robot description, URDF)
Before this commit: robot Robot_Arm, 7 links, 6 joints
Joints:
- joint Gripper_left: origin xyz=-0.0175 0.015 0.064 rpy=0 0 0 -> xyz=-0.0175 0.015 0.064 rpy=-1.57 0 0
- joint Gripper_right: origin xyz=-0.0175 -0.015 0.064 rpy=0 0 0 -> xyz=-0.0175 -0.015 0.064 rpy=1.57 0 0

Commit message: Modify : Reconstruct the framework of RobotArm.

File: urdf/Robot_Arm.urdf (robot description, URDF)
Before this commit: robot Robot_Arm, 7 links, 6 joints
Links:
- added link Arm_Base
- added link Camera
Joints:
- added joint Arm_Locate: type fixed, parent world, child Arm_Base, origin xyz=0.0 0.2 0.0 rpy=0.0 0.0 0.0
- added joint Camera_Locate: type fixed, parent arm_link_1, child Camera, origin xyz=0.0 -0.02 0.2 rpy=3.14 0.5 0
- joint arm_joint_1: parent world -> Arm_Base
